File: back/back.kicad_pcb (KiCad board)
At the start: 2 copper layers, 57.5 x 48.8 mm, 16 parts, among them J1 Screw_Terminal_01x02, J2 Screw_Terminal_01x02, Q1 IRF510, U1 NE555

Commit message: Schema final
Parts:
- added J3: Screw_Terminal_01x02, TerminalBlock_4Ucon:TerminalBlock_4Ucon_1x02_P3.50mm_Vertical, F.Cu at (138.0, 89.0)
- C4: value 10n -> 820p
- D1: value D -> D_x2_KCom_KAA; footprint Diode_THT:D_DO-34_SOD68_P10.16mm_Horizontal -> Package_TO_SOT_THT:TO-220-3_Vertical
- L1: footprint Inductor_THT:L_Radial_D21.0mm_P14.61mm_Vishay_IHB-2 -> back:ind_W60mm_D19mm_P38mm
- moved J2 88.7 mm to (193.0, 69.0), turned to 270 degrees
- moved C1 71.0 mm to (185.0, 69.0), turned to 180 degrees
- moved C2 69.2 mm to (185.0, 77.0)
- moved R1 68.2 mm to (128.0, 68.0), turned to 270 degrees
- moved Q1 64.9 mm to (133.0, 63.0)
- moved R3 61.0 mm to (156.0, 72.0)
- moved C4 60.9 mm to (161.0, 77.0), turned to 0 degrees
- moved U1 60.5 mm to (133.0, 73.0), turned to 0 degrees
- moved R4 59.6 mm to (146.0, 76.0), turned to 0 degrees
- moved D3 59.4 mm to (146.0, 79.0), turned to 0 degrees
- moved J1 59.3 mm to (121.0, 60.0), turned to 90 degrees
- moved D2 59.0 mm to (156.0, 68.0)
- moved R2 55.0 mm to (143.0, 68.0)
- moved L1 51.6 mm to (148.0, 58.0), turned to 0 degrees
- moved D1 49.2 mm to (133.0, 49.0)
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Connections:
- C1 pad 1: +12V -> Net-(C1-Pad1)
- C2 pad 1: +12V -> Net-(C1-Pad1)
- D1 pad 1: Net-(D1-Pad1) -> /GNDCLK
- D3 pad 1: Net-(D3-Pad1) -> Net-(D2-Pad2)
- J2 pad 1: +12V -> Net-(C1-Pad1)
- L1 pad 1: Net-(D1-Pad1) -> /GNDCLK
- L1 pad 2: +12V -> Net-(C1-Pad1)
- Q1 pad 3: Net-(D1-Pad1) -> /GNDCLK
- R2 pad 2: +12V -> /RST
- U1 pad 1: GND -> /GNDCLK
- U1 pad 4: +12V -> /RST
- U1 pad 7: Net-(D3-Pad1) -> Net-(D2-Pad2)
- U1 pad 8: +12V -> /RST
Routing:
- net GND: track 85.9 -> 0.00 mm
- net +12V: track 60.0 -> 0.00 mm
- net /TRIG: track 34.7 -> 0.00 mm
- net Net-(D1-Pad1): track 26.4 -> 0.00 mm
- net Net-(J1-Pad2): track 14.6 -> 0.00 mm
- net Net-(Q1-Pad1): track 8.08 -> 0.00 mm
- net /Q_Base: track 7.59 -> 0.00 mm
- net Net-(D3-Pad1): track 7.22 -> 0.00 mm
- net Net-(D2-Pad2): track 7.02 -> 0.00 mm
- net Net-(D2-Pad1): track 6.00 -> 0.00 mm
- net Net-(C3-Pad1): track 4.74 -> 0.00 mm
- net Net-(D3-Pad2): track 2.75 -> 0.00 mm
- removed copper zone on F.Cu, net GND
Other:
- board size 57.5 x 48.8 mm -> 89 x 45 mm

Commit message: Final version v2
Parts:
- moved J2 52.5 mm to (156.5, 106.8), turned to 180 degrees
- moved D1 38.4 mm to (170.0, 59.2)
- moved R1 35.6 mm to (158.8, 50.0)
- moved C2 34.5 mm to (160.8, 101.5), turned to 0 degrees
- moved Q1 33.7 mm to (164.8, 51.8), turned to 0 degrees
- moved L1 33.3 mm to (181.2, 57.8), turned to 270 degrees
- moved J1 31.3 mm to (149.8, 47.8), turned to 0 degrees
- moved C1 30.1 mm to (170.8, 95.5)
- moved J3 29.7 mm to (151.0, 62.2), turned to 90 degrees
- moved R2 29.5 mm to (172.5, 67.2)
- moved U1 26.1 mm to (158.5, 67.5), turned to 270 degrees
- moved D3 24.8 mm to (170.8, 78.2), turned to 270 degrees
- moved R3 17.7 mm to (167.1, 85.8), turned to 90 degrees
- moved R4 17.1 mm to (163.1, 75.8), turned to 270 degrees
- moved C3 8.14 mm to (152.0, 78.5), turned to 270 degrees
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Routing:
- net /GNDCLK: track 0.00 -> 34.7 mm
- net Net-(D2-Pad2): track 0.00 -> 34.6 mm
- net Net-(C1-Pad1): track 0.00 -> 31.8 mm
- net /RST: track 0.00 -> 30.3 mm
- net /Q_Base: track 0.00 -> 29.3 mm
- net /TRIG: track 0.00 -> 25.9 mm
- net Net-(D2-Pad1): track 0.00 -> 18.6 mm
- net Net-(J1-Pad2): track 0.00 -> 17.9 mm
- net Net-(D3-Pad2): track 0.00 -> 8.64 mm
- net Net-(Q1-Pad1): track 0.00 -> 6.72 mm
- net Net-(C3-Pad1): track 0.00 -> 3.84 mm
- added copper zone on F.Cu, net GND
Other:
- board size 89 x 45 mm -> 65 x 70 mm
- net class Power: clearance 0.2 -> 0.4

Commit message: zajecia
Parts:
- removed R3: 40k, Resistor_THT:R_Axial_DIN0207_L6.3mm_D2.5mm_P10.16mm_Horizontal
- removed R4: 10k, Resistor_THT:R_Axial_DIN0207_L6.3mm_D2.5mm_P10.16mm_Horizontal
- added REF**: MountingHole_2.5mm, MountingHole:MountingHole_2.5mm, F.Cu at (142.5, 47.5)
- added REF**: MountingHole_2.5mm, MountingHole:MountingHole_2.5mm, F.Cu at (142.5, 107.5)
- added REF**: MountingHole_2.5mm, MountingHole:MountingHole_2.5mm, F.Cu at (197.5, 107.5)
- added REF**: MountingHole_2.5mm, MountingHole:MountingHole_2.5mm, F.Cu at (197.5, 47.5)
- added RV1: R_POT_TRIM, Potentiometer_THT:Potentiometer_Piher_PT-10-V10_Vertical, F.Cu at (162.5, 79.1)
- C3: value 10n -> 100n
- C4: footprint Capacitor_THT:C_Disc_D7.5mm_W5.0mm_P10.00mm -> Capacitor_SMD:C_0603_1608Metric_Pad1.05x0.95mm_HandSolder
- moved C4 3.78 mm to (158.5, 82.2)
- moved D3 1.27 mm to (172.0, 78.0)
- moved D2 1.25 mm to (162.2, 73.0)
Routing:
- net /TRIG: track 25.9 -> 64.0 mm
- net (no net): track 0.00 -> 36.4 mm
- net /Q_Base: track 29.3 -> 9.95 mm
- net Net-(D2-Pad1): track 18.6 -> 6.15 mm
- net /RST: track 30.3 -> 24.1 mm
- net GND: track 0.00 -> 5.75 mm, vias 0 -> 2
- net Net-(D3-Pad2): track 8.64 -> 11.0 mm
- net Net-(D2-Pad2): track 34.6 -> 35.8 mm
Other:
- net class Default: clearance 0.2 -> 0.5; trace_width 0.3 -> 1
- net class Power: clearance 0.4 -> 0.5; trace_width 1 -> 1.5
- rule trace_clearance: 0.2 -> 0.5

Commit message: wersja nie dzialajaca
Parts:
- U1: footprint Package_DIP:DIP-8_W7.62mm_LongPads -> Package_DIP:DIP-8_W10.16mm_LongPads
- moved C3 7.42 mm to (146.8, 83.8)
- moved C4 3.88 mm to (158.5, 86.1)
- moved U1 2.80 mm to (156.0, 68.8)
Routing:
- net /RST: track 24.1 -> 43.9 mm
- net Net-(C3-Pad1): track 3.84 -> 20.8 mm
- net (no net): track 36.4 -> 21.1 mm
- net /TRIG: track 64.0 -> 70.5 mm
- net /GNDCLK: track 35.1 -> 38.1 mm
- net /Q_Base: track 9.95 -> 12.7 mm
- net Net-(D2-Pad2): track 35.8 -> 34.4 mm

Commit message: final 6.10
Parts:
- removed REF** (x4): MountingHole_2.5mm, MountingHole:MountingHole_2.5mm
- C1: value 1u -> 22u
- J1, J2, J3: footprint TerminalBlock_4Ucon:TerminalBlock_4Ucon_1x02_P3.50mm_Vertical -> TerminalBlock:TerminalBlock_bornier-2_P5.08mm
- L1: footprint back:ind_W60mm_D19mm_P38mm -> Footprints:ind_W60mm_D19mm_P38mm
- moved J1 91.4 mm to (81.5, 108.5), turned to 90 degrees
- moved R1 78.2 mm to (94.2, 94.2), turned to 90 degrees
- moved Q1 77.3 mm to (106.0, 102.0), turned to 90 degrees
- moved D1 62.4 mm to (125.8, 103.2), turned to 0 degrees
- moved RV1 54.4 mm to (111.0, 61.5), turned to 0 degrees
- moved J2 51.5 mm to (113.0, 134.2)
- moved D2 50.6 mm to (111.8, 69.2)
- moved D3 50.2 mm to (122.0, 73.0), turned to 180 degrees
- moved R2 48.5 mm to (124.0, 66.2)
- moved U1 40.7 mm to (119.5, 86.8), turned to 90 degrees
- moved C1 40.0 mm to (139.5, 120.5)
- moved C2 37.2 mm to (139.5, 132.0), turned to 180 degrees
- moved L1 33.1 mm to (155.5, 78.5)
- moved C4 26.3 mm to (137.5, 70.2), turned to 0 degrees
- moved C3 13.4 mm to (133.8, 80.5), turned to 0 degrees
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Connections:
- C3 pad 2: GND -> /GNDCLK
- C4 pad 2: GND -> /GNDCLK
- J3 pad 2: GND -> /GNDCLK
Routing:
- net /GNDCLK: track 38.1 -> 157.9 mm
- net (no net): track 21.1 -> 100.4 mm
- net Net-(C1-Pad1): track 31.8 -> 61.0 mm
- net Net-(D2-Pad2): track 34.4 -> 11.3 mm
- net /Q_Base: track 12.7 -> 33.8 mm
- net Net-(J1-Pad2): track 17.9 -> 34.9 mm
- net /RST: track 43.9 -> 59.8 mm
- net Net-(C3-Pad1): track 20.8 -> 8.25 mm
- net /TRIG: track 70.5 -> 58.5 mm
- net Net-(D3-Pad2): track 11.0 -> 20.6 mm
- net Net-(Q1-Pad1): track 6.72 -> 15.0 mm
- net GND: track 5.75 -> 0.00 mm, vias 2 -> 0
- net Net-(D2-Pad1): track 6.15 -> 8.06 mm
Other:
- board size 65 x 70 mm -> 100 x 98.8 mm
- net class Default: trace_width 1 -> 1.5; via_dia 0.8 -> 1; via_drill 0.4 -> 0.5
- net class Power: trace_width 1.5 -> 2; via_dia 0.8 -> 1.5; via_drill 0.4 -> 0.5
