File: back/back.sch (KiCad schematic (older format))
At the start: 11 parts

Commit message: schematic ideal
Parts:
- added C?: C, symbol Device:C
- added L?: L, symbol Device:L
Connections:
- net labels added: TRIG
- wire segments 25 -> 43
Other:
- moved on the sheet: C?, R?
Changed lines of the file:
@@
 	3150 950  3150 1050
 Wire Wire Line
-	3150 950  3800 950
+	3150 950  3350 950
 Wire Wire Line
 	3800 950  3800 1050
@@
 Wire Wire Line
 	2850 2700 2850 3100
-$Comp
-L Device:C C?
-U 1 1 5CB1966A
-P 1500 3450
-F 0 "C?" H 1615 3496 50  0000 L CNN
-F 1 "C" H 1615 3405 50  0000 L CNN
-F 2 "" H 1538 3300 50  0001 C CNN
-F 3 "~" H 1500 3450 50  0001 C CNN
-	1    1500 3450
-	1    0    0    -1
-$EndComp
-$Comp
-L power:GND #PWR?
-U 1 1 5CB1D636
-P 1500 3950
-F 0 "#PWR?" H 1500 3700 50  0001 C CNN
-F 1 "GND" H 1505 3777 50  0000 C CNN
-F 2 "" H 1500 3950 50  0001 C CNN
-F 3 "" H 1500 3950 50  0001 C CNN
-	1    1500 3950
-	1    0    0    -1
-$EndComp
-Wire Wire Line
-	1500 3600 1500 3950
-Wire Wire Line
-	1500 3100 1500 3300
-$Comp
-L Device:R R?
-U 1 1 5CB1E3D7
-P 1800 3800
-F 0 "R?" H 1870 3846 50  0000 L CNN
-F 1 "R" H 1870 3755 50  0000 L CNN
-F 2 "" V 1730 3800 50  0001 C CNN
-F 3 "~" H 1800 3800 50  0001 C CNN
-	1    1800 3800
-	1    0    0    -1
-$EndComp
-$Comp
-L Device:R R?
-U 1 1 5CB1EF33
-P 1800 3400
-F 0 "R?" H 1870 3446 50  0000 L CNN
-F 1 "R" H 1870 3355 50  0000 L CNN
-F 2 "" V 1730 3400 50  0001 C CNN
-F 3 "~" H 1800 3400 50  0001 C CNN
-	1    1800 3400
-	1    0    0    -1
-$EndComp
 Wire Wire Line
 	2650 3100 2850 3100
@@
 L power:+5V #PWR?
 U 1 1 5CB21EF9
-P 1500 3100
-F 0 "#PWR?" H 1500 2950 50  0001 C CNN
-F 1 "+5V" H 1515 3273 50  0000 C CNN
-F 2 "" H 1500 3100 50  0001 C CNN
-F 3 "" H 1500 3100 50  0001 C CNN
-	1    1500 3100
-	1    0    0    -1
-$EndComp
+P 4450 2650
+F 0 "#PWR?" H 4450 2500 50  0001 C CNN
+F 1 "+5V" H 4465 2823 50  0000 C CNN
+F 2 "" H 4450 2650 50  0001 C CNN
+F 3 "" H 4450 2650 50  0001 C CNN
+	1    4450 2650
+	1    0    0    -1
+$EndComp
+Connection ~ 4450 3000
+Wire Wire Line
+	4150 3000 4450 3000
+Wire Wire Line
+	4150 3100 4150 3000
+Wire Wire Line
+	4150 3500 4150 3400
+$Comp
+L power:GND #PWR?
+U 1 1 5CB2275D
+P 4150 4100
+F 0 "#PWR?" H 4150 3850 50  0001 C CNN
+F 1 "GND" H 4155 3927 50  0000 C CNN
+F 2 "" H 4150 4100 50  0001 C CNN
+F 3 "" H 4150 4100 50  0001 C CNN
+	1    4150 4100
+	1    0    0    -1
+$EndComp
+$Comp
+L Device:R R?
+U 1 1 5CB1EF33
+P 4150 3250
+F 0 "R?" H 4220 3296 50  0000 L CNN
+F 1 "R" H 4220 3205 50  0000 L CNN
+F 2 "" V 4080 3250 50  0001 C CNN
+F 3 "~" H 4150 3250 50  0001 C CNN
+	1    4150 3250
+	1    0    0    -1
+$EndComp
+$Comp
+L Device:R R?
+U 1 1 5CB1E3D7
+P 4150 3750
+F 0 "R?" H 4220 3796 50  0000 L CNN
+F 1 "R" H 4220 3705 50  0000 L CNN
+F 2 "" V 4080 3750 50  0001 C CNN
+F 3 "~" H 4150 3750 50  0001 C CNN
+	1    4150 3750
+	1    0    0    -1
+$EndComp
+$Comp
+L power:GND #PWR?
+U 1 1 5CB1D636
+P 4450 4100
+F 0 "#PWR?" H 4450 3850 50  0001 C CNN
+F 1 "GND" H 4455 3927 50  0000 C CNN
+F 2 "" H 4450 4100 50  0001 C CNN
+F 3 "" H 4450 4100 50  0001 C CNN
+	1    4450 4100
+	1    0    0    -1
+$EndComp
+$Comp
+L Device:C C?
+U 1 1 5CB1966A
+P 4450 3550
+F 0 "C?" H 4565 3596 50  0000 L CNN
+F 1 "C" H 4565 3505 50  0000 L CNN
+F 2 "" H 4488 3400 50  0001 C CNN
+F 3 "~" H 4450 3550 50  0001 C CNN
+	1    4450 3550
+	1    0    0    -1
+$EndComp
+Wire Wire Line
+	4450 2650 4450 3000
+Wire Wire Line
+	3150 3500 4150 3500
+Wire Wire Line
+	4150 3500 4150 3600
+Connection ~ 4150 3500
+Wire Wire Line
+	3150 3700 3950 3700
+Wire Wire Line
+	3950 3700 3950 4000
+Wire Wire Line
+	3950 4000 4150 4000
+Wire Wire Line
+	4150 4000 4150 3900
+Wire Wire Line
+	4150 4000 4150 4100
+Connection ~ 4150 4000
+Wire Wire Line
+	4450 3700 4450 4100
+Wire Wire Line
+	4450 3000 4450 3400
+Wire Wire Line
+	4150 3000 3950 3000
+Connection ~ 4150 3000
+Text Label 3950 3000 0    50   ~ 0
+TRIG
+Wire Wire Line
+	2150 3300 1950 3300
+Text Label 1950 3300 0    50   ~ 0
+TRIG
+$Comp
+L Device:C C?
+U 1 1 5CB37AF6
+P 1600 3650
+F 0 "C?" H 1715 3696 50  0000 L CNN
+F 1 "C" H 1715 3605 50  0000 L CNN
+F 2 "" H 1638 3500 50  0001 C CNN
+F 3 "~" H 1600 3650 50  0001 C CNN
+	1    1600 3650
+	1    0    0    -1
+$EndComp
+Wire Wire Line
+	2150 3500 1600 3500
+$Comp
+L power:GND #PWR?
+U 1 1 5CB39283
+P 1600 3950
+F 0 "#PWR?" H 1600 3700 50  0001 C CNN
+F 1 "GND" H 1605 3777 50  0000 C CNN
+F 2 "" H 1600 3950 50  0001 C CNN
+F 3 "" H 1600 3950 50  0001 C CNN
+	1    1600 3950
+	1    0    0    -1
+$EndComp
+Wire Wire Line
+	1600 3800 1600 3950
+$Comp
+L power:+5V #PWR?
+U 1 1 5CB3AAE4
+P 2050 3950
+F 0 "#PWR?" H 2050 3800 50  0001 C CNN
+F 1 "+5V" H 2065 4123 50  0000 C CNN
+F 2 "" H 2050 3950 50  0001 C CNN
+F 3 "" H 2050 3950 50  0001 C CNN
+	1    2050 3950
+	-1   0    0    1
+$EndComp
+Wire Wire Line
+	2150 3700 2050 3700
+Wire Wire Line
+	2050 3700 2050 3950
+$Comp
+L Device:L L?
+U 1 1 5CB3BF6E
+P 3500 950
+F 0 "L?" V 3690 950 50  0000 C CNN
+F 1 "L" V 3599 950 50  0000 C CNN
+F 2 "" H 3500 950 50  0001 C CNN
+F 3 "~" H 3500 950 50  0001 C CNN
+	1    3500 950
+	0    -1   -1   0
+$EndComp
+Wire Wire Line
+	3650 950  3800 950
 $EndSCHEMATC

Commit message: final v1
Parts:
- removed J? (x2): Conn_01x01, symbol Connector_Generic:Conn_01x01
- removed Q?: 2N2219, Package_TO_SOT_THT:TO-39-3, symbol Transistor_BJT:2N2219
- removed R?: R, symbol Device:R
- added D2, D3: D, Diode_THT:D_DO-34_SOD68_P10.16mm_Horizontal, symbol Device:D
- added J1, J2: Screw_Terminal_01x02, TerminalBlock_4Ucon:TerminalBlock_4Ucon_1x02_P3.50mm_Vertical, symbol Connector:Screw_Terminal_01x02
- added Q1: IRF510, Package_TO_SOT_THT:TO-220-3_Vertical, symbol Transistor_FET:IRF540N
- added R1: 330, Resistor_THT:R_Axial_DIN0207_L6.3mm_D2.5mm_P10.16mm_Horizontal, symbol Device:R
- added R2: 1k, Resistor_THT:R_Axial_DIN0207_L6.3mm_D2.5mm_P10.16mm_Horizontal, symbol Device:R
- C1: renamed from C?; value C -> 1u; footprint (none) -> Capacitor_THT:CP_Axial_L11.0mm_D5.0mm_P18.00mm_Horizontal
- C2: renamed from C?; value C -> 100n; footprint (none) -> Capacitor_THT:C_Disc_D7.5mm_W5.0mm_P10.00mm
- C3, C4: renamed from C?; value C -> 10n; footprint (none) -> Capacitor_THT:C_Disc_D7.5mm_W5.0mm_P10.00mm
- D1: renamed from D?; footprint (none) -> Diode_THT:D_DO-34_SOD68_P10.16mm_Horizontal
- L1: renamed from L?; value L -> 400u; footprint (none) -> Inductor_THT:L_Radial_D21.0mm_P14.61mm_Vishay_IHB-2
- R3: renamed from R?; value R -> 40k; footprint (none) -> Resistor_THT:R_Axial_DIN0207_L6.3mm_D2.5mm_P10.16mm_Horizontal
- R4: renamed from R?; value R -> 10k; footprint (none) -> Resistor_THT:R_Axial_DIN0207_L6.3mm_D2.5mm_P10.16mm_Horizontal
- U1: renamed from U?; footprint (none) -> Package_DIP:DIP-8_W7.62mm_LongPads
Connections:
- net labels added: +12V
- net labels removed: +24V, +5V
- wire segments 43 -> 52
Other:
- note added: "Układ przetwarzający"
- note added: "Układ zegarowy"
- moved on the sheet: C1, C2, C3, C4, D1, L1, R3, R4, U1

Commit message: Schema final
Parts:
- removed D1: D, Diode_THT:D_DO-34_SOD68_P10.16mm_Horizontal, symbol Device:D
- added D1: D_x2_KCom_KAA, Package_TO_SOT_THT:TO-220-3_Vertical, symbol Device:D_x2_KCom_KAA
- added J3: Screw_Terminal_01x02, TerminalBlock_4Ucon:TerminalBlock_4Ucon_1x02_P3.50mm_Vertical, symbol Connector:Screw_Terminal_01x02
- C4: value 10n -> 820p
- L1: footprint Inductor_THT:L_Radial_D21.0mm_P14.61mm_Vishay_IHB-2 -> back:ind_W60mm_D19mm_P38mm
Connections:
- net GND: now also D1.2 (A), D1.3 (A), J3.2 (Pin_2); no longer U1.1 (GND)
- net GNDCLK: now reaches L1.1, Q1.3 (S)
- net GNDCLK: now also U1.1 (GND), D1.1 (K)
- net at D3.1 (K), U1.7 (DIS): now also D2.2 (A), R2.1
- net +12V: no longer names the net of C1.1, C2.1, J2.1 (Pin_1), L1.2
- net +12V: no longer R2.2, U1.4 (R), U1.8 (VCC)
- new net RST: J3.1 (Pin_1), R2.2, U1.4 (R), U1.8 (VCC)
Other:
- moved on the sheet: C1, C2, J2, L1
Changed lines of the file:
@@
 EESchema Schematic File Version 4
 LIBS:back-cache
-EELAYER 26 0
+EELAYER 29 0
 EELAYER END
 $Descr A4 11693 8268
@@
 L power:GND #PWR0101
 U 1 1 5CB04671
-P 3800 1950
-F 0 "#PWR0101" H 3800 1700 50  0001 C CNN
-F 1 "GND" H 3805 1777 50  0000 C CNN
-F 2 "" H 3800 1950 50  0001 C CNN
-F 3 "" H 3800 1950 50  0001 C CNN
-	1    3800 1950
-	1    0    0    -1
-$EndComp
-$Comp
-L Device:D D1
-U 1 1 5CB0ACC5
-P 3150 1750
-F 0 "D1" V 3104 1829 50  0000 L CNN
-F 1 "D" V 3195 1829 50  0000 L CNN
-F 2 "Diode_THT:D_DO-34_SOD68_P10.16mm_Horizontal" H 3150 1750 50  0001 C CNN
-F 3 "~" H 3150 1750 50  0001 C CNN
-	1    3150 1750
-	0    1    1    0
+P 4100 1850
+F 0 "#PWR0101" H 4100 1600 50  0001 C CNN
+F 1 "GND" H 4105 1677 50  0000 C CNN
+F 2 "" H 4100 1850 50  0001 C CNN
+F 3 "" H 4100 1850 50  0001 C CNN
+	1    4100 1850
+	1    0    0    -1
 $EndComp
 $Comp
 L Device:C C1
 U 1 1 5CB0B470
-P 3800 1750
-F 0 "C1" H 3915 1796 50  0000 L CNN
-F 1 "1u" H 3915 1705 50  0000 L CNN
-F 2 "Capacitor_THT:CP_Axial_L11.0mm_D5.0mm_P18.00mm_Horizontal" H 3838 1600 50  0001 C CNN
-F 3 "~" H 3800 1750 50  0001 C CNN
-	1    3800 1750
+P 4100 1650
+F 0 "C1" H 4215 1696 50  0000 L CNN
+F 1 "1u" H 4215 1605 50  0000 L CNN
+F 2 "Capacitor_THT:CP_Axial_L11.0mm_D5.0mm_P18.00mm_Horizontal" H 4138 1500 50  0001 C CNN
+F 3 "~" H 4100 1650 50  0001 C CNN
+	1    4100 1650
 	1    0    0    -1
 $EndComp
@@
 L Device:C C2
 U 1 1 5CB0DCF7
-P 4300 1750
-F 0 "C2" H 4415 1796 50  0000 L CNN
-F 1 "100n" H 4415 1705 50  0000 L CNN
-F 2 "Capacitor_THT:C_Disc_D7.5mm_W5.0mm_P10.00mm" H 4338 1600 50  0001 C CNN
-F 3 "~" H 4300 1750 50  0001 C CNN
-	1    4300 1750
-	1    0    0    -1
-$EndComp
-Wire Wire Line
-	3150 1900 3150 1950
-Wire Wire Line
-	2900 1500 3150 1500
-Wire Wire Line
-	3150 1500 3150 1600
-Wire Wire Line
-	3150 1500 3350 1500
-Wire Wire Line
-	3800 1500 3800 1600
-Connection ~ 3150 1500
-Wire Wire Line
-	3150 1950 3800 1950
-Wire Wire Line
-	3800 1950 3800 1900
-Wire Wire Line
-	3800 1950 4300 1950
-Wire Wire Line
-	4300 1950 4300 1900
-Connection ~ 3800 1950
-Wire Wire Line
-	4300 1500 4300 1600
-Connection ~ 3800 1500
-Connection ~ 4300 1500
-Wire Wire Line
-	3800 1500 4300 1500
-Wire Wire Line
-	4500 1350 4500 1500
-Connection ~ 4500 1500
-Wire Wire Line
-	4500 1500 4300 1500
+P 4600 1650
+F 0 "C2" H 4715 1696 50  0000 L CNN
+F 1 "100n" H 4715 1605 50  0000 L CNN
+F 2 "Capacitor_THT:C_Disc_D7.5mm_W5.0mm_P10.00mm" H 4638 1500 50  0001 C CNN
+F 3 "~" H 4600 1650 50  0001 C CNN
+	1    4600 1650
+	1    0    0    -1
+$EndComp
+Wire Wire Line
+	4100 1400 4100 1500
+Wire Wire Line
+	4100 1850 4100 1800
+Wire Wire Line
+	4100 1850 4600 1850
+Wire Wire Line
+	4600 1850 4600 1800
+Connection ~ 4100 1850
+Wire Wire Line
+	4600 1400 4600 1500
+Connection ~ 4100 1400
+Connection ~ 4600 1400
+Wire Wire Line
+	4100 1400 4600 1400
 Text Label 3100 4650 0    50   ~ 0
 Q_Base
@@
 Wire Wire Line
 	2350 5250 2350 5350
-$Comp
-L power:GND #PWR0102
-U 1 1 5CB126F3
-P 2350 5350
-F 0 "#PWR0102" H 2350 5100 50  0001 C CNN
-F 1 "GND" H 2355 5177 50  0000 C CNN
-F 2 "" H 2350 5350 50  0001 C CNN
-F 3 "" H 2350 5350 50  0001 C CNN
-	1    2350 5350
-	1    0    0    -1
-$EndComp
-Wire Wire Line
-	2550 4050 2550 4450
 Wire Wire Line
 	2350 4450 2550 4450
@@
 P 3650 5350
 F 0 "C4" H 3765 5396 50  0000 L CNN
-F 1 "10n" H 3765 5305 50  0000 L CNN
+F 1 "820p" H 3765 5305 50  0000 L CNN
 F 2 "Capacitor_THT:C_Disc_D7.5mm_W5.0mm_P10.00mm" H 3688 5200 50  0001 C CNN
 F 3 "~" H 3650 5350 50  0001 C CNN
@@
 Wire Wire Line
 	1850 5050 1750 5050
-Wire Wire Line
-	1750 5050 1750 5300
 $Comp
 L Device:L L1
 U 1 1 5CB3BF6E
-P 3500 1500
-F 0 "L1" V 3690 1500 50  0000 C CNN
-F 1 "400u" V 3599 1500 50  0000 C CNN
-F 2 "Inductor_THT:L_Radial_D21.0mm_P14.61mm_Vishay_IHB-2" H 3500 1500 50  0001 C CNN
-F 3 "~" H 3500 1500 50  0001 C CNN
-	1    3500 1500
+P 3800 1400
+F 0 "L1" V 3990 1400 50  0000 C CNN
+F 1 "400u" V 3899 1400 50  0000 C CNN
+F 2 "back:ind_W60mm_D19mm_P38mm" H 3800 1400 50  0001 C CNN
+F 3 "~" H 3800 1400 50  0001 C CNN
+	1    3800 1400
 	0    -1   -1   0
 $EndComp
 Wire Wire Line
-	3650 1500 3800 1500
+	3950 1400 4100 1400
 $Comp
 L Device:R R1
@@
 Wire Wire Line
 	2700 1800 2700 1950
-Wire Wire Line
-	1300 1500 2500 1500
 $Comp
 L Connector:Screw_Terminal_01x02 J2
 U 1 1 5CC2AE89
-P 4950 1700
-F 0 "J2" H 5030 1692 50  0000 L CNN
-F 1 "Screw_Terminal_01x02" H 5030 1601 50  0000 L CNN
-F 2 "TerminalBlock_4Ucon:TerminalBlock_4Ucon_1x02_P3.50mm_Vertical" H 4950 1700 50  0001 C CNN
-F 3 "~" H 4950 1700 50  0001 C CNN
-	1    4950 1700
-	1    0    0    -1
-$EndComp
-Wire Wire Line
-	4750 1500 4750 1700
-Wire Wire Line
-	4500 1500 4750 1500
-Wire Wire Line
-	4750 1800 4750 1950
-Wire Wire Line
-	4750 1950 4300 1950
-Connection ~ 4300 1950
+P 5250 1600
+F 0 "J2" H 5330 1592 50  0000 L CNN
+F 1 "Screw_Terminal_01x02" H 5330 1501 50  0000 L CNN
+F 2 "TerminalBlock_4Ucon:TerminalBlock_4Ucon_1x02_P3.50mm_Vertical" H 5250 1600 50  0001 C CNN
+F 3 "~" H 5250 1600 50  0001 C CNN
+	1    5250 1600
+	1    0    0    -1
+$EndComp
+Wire Wire Line
+	5050 1400 5050 1600
+Wire Wire Line
+	5050 1700 5050 1850
+Wire Wire Line
+	5050 1850 4600 1850
+Connection ~ 4600 1850
 $Comp
 L Connector:Screw_Terminal_01x02 J1
@@
 	0    -1   -1   0
 $EndComp
-$Comp
-L power:+12V #PWR0106
-U 1 1 5CC2EC30
-P 3000 3550
-F 0 "#PWR0106" H 3000 3400 50  0001 C CNN
-F 1 "+12V" H 3015 3723 50  0000 C CNN
-F 2 "" H 3000 3550 50  0001 C CNN
-F 3 "" H 3000 3550 50  0001 C CNN
-	1    3000 3550
-	1    0    0    -1
-$EndComp
-$Comp
-L power:+12V #PWR0107
-U 1 1 5CC2EC6C
-P 4500 1350
-F 0 "#PWR0107" H 4500 1200 50  0001 C CNN
-F 1 "+12V" H 4515 1523 50  0000 C CNN
-F 2 "" H 4500 1350 50  0001 C CNN
-F 3 "" H 4500 1350 50  0001 C CNN
-	1    4500 1350
-	1    0    0    -1
-$EndComp
-$Comp
-L power:+12V #PWR0108
-U 1 1 5CC2ED75
-P 2550 4050
-F 0 "#PWR0108" H 2550 3900 50  0001 C CNN
-F 1 "+12V" H 2565 4223 50  0000 C CNN
-F 2 "" H 2550 4050 50  0001 C CNN
-F 3 "" H 2550 4050 50  0001 C CNN
-	1    2550 4050
-	1    0    0    -1
-$EndComp
-$Comp
-L power:+12V #PWR0109
-U 1 1 5CC2EDBF
-P 1750 5300
-F 0 "#PWR0109" H 1750 5150 50  0001 C CNN
-F 1 "+12V" H 1765 5473 50  0000 C CNN
-F 2 "" H 1750 5300 50  0001 C CNN
-F 3 "" H 1750 5300 50  0001 C CNN
-	1    1750 5300
-	-1   0    0    1
-$EndComp
 Wire Wire Line
 	3650 5050 3650 5200
@@
 	4150 3850 4050 3850
 Wire Wire Line
-	3000 3550 3000 3850
-Wire Wire Line
 	4450 4350 4450 4200
 Wire Wire Line
@@
 	0    1    1    0
 $EndComp
-Wire Wire Line
-	3000 3850 3150 3850
 Text Notes 1400 850  0    50   ~ 0
 Układ przetwarzający
@@
 Układ zegarowy
 Wire Wire Line
-	3450 3850 3750 3850
-Wire Wire Line
-	2850 4850 3750 4850
+	3450 3850 3600 3850
+Wire Wire Line
+	2850 4850 3600 4850
+$Comp
+L Connector:Screw_Terminal_01x02 J3
+U 1 1 5CC30FEE
+P 2550 3400
+F 0 "J3" V 2514 3212 50  0000 R CNN
+F 1 "Screw_Terminal_01x02" V 2423 3212 50  0000 R CNN
+F 2 "TerminalBlock_4Ucon:TerminalBlock_4Ucon_1x02_P3.50mm_Vertical" H 2550 3400 50  0001 C CNN
+F 3 "~" H 2550 3400 50  0001 C CNN
+	1    2550 3400
+	0    -1   -1   0
+$EndComp
+Wire Wire Line
+	2550 3600 2550 3850
+$Comp
+L Device:D_x2_KCom_KAA D1
+U 1 1 5CC355F8
+P 3250 1700
+F 0 "D1" H 3200 1800 50  0000 L CNN
+F 1 "D_x2_KCom_KAA" H 2950 1950 50  0000 L CNN
+F 2 "Package_TO_SOT_THT:TO-220-3_Vertical" H 3250 1700 50  0001 C CNN
+F 3 "~" H 3250 1700 50  0001 C CNN
+	1    3250 1700
+	-1   0    0    1
+$EndComp
+Wire Wire Line
+	2900 1500 2950 1500
+Wire Wire Line
+	3650 1500 3650 1400
+Wire Wire Line
+	4600 1400 5050 1400
+Wire Wire Line
+	2950 1500 2950 1300
+Text Label 2950 1300 0    50   ~ 0
+GNDCLK
+Text Label 2350 5350 0    50   ~ 0
+GNDCLK
+Wire Wire Line
+	1300 1500 2500 1500
+Connection ~ 2950 1500
+Connection ~ 2550 3850
+Wire Wire Line
+	2550 3850 2550 4450
+Wire Wire Line
+	2550 3850 2250 3850
+Text Label 2250 3850 0    50   ~ 0
+RST
+Text Label 1750 5350 0    50   ~ 0
+RST
+Wire Wire Line
+	2650 3600 2850 3600
+Wire Wire Line
+	1750 5050 1750 5350
+Wire Wire Line
+	3600 3850 3600 4850
+Connection ~ 3600 3850
+Wire Wire Line
+	3600 3850 3750 3850
+Connection ~ 3600 4850
+Wire Wire Line
+	3600 4850 3750 4850
+$Comp
+L power:GND #PWR0102
+U 1 1 5CC493B4
+P 2850 3600
+F 0 "#PWR0102" H 2850 3350 50  0001 C CNN
+F 1 "GND" H 2855 3427 50  0000 C CNN
+F 2 "" H 2850 3600 50  0001 C CNN
+F 3 "" H 2850 3600 50  0001 C CNN
+	1    2850 3600
+	1    0    0    -1
+$EndComp
+$Comp
+L power:GND #PWR0106
+U 1 1 5CC5B78A
+P 3650 1700
+F 0 "#PWR0106" H 3650 1450 50  0001 C CNN
+F 1 "GND" V 3655 1572 50  0000 R CNN
+F 2 "" H 3650 1700 50  0001 C CNN
+F 3 "" H 3650 1700 50  0001 C CNN
+	1    3650 1700
+	0    -1   -1   0
+$EndComp
+Wire Wire Line
+	2950 1500 3250 1500
+Wire Wire Line
+	2950 1700 2950 1850
+Wire Wire Line
+	2950 1850 4100 1850
+Wire Wire Line
+	3550 1700 3650 1700
+Wire Wire Line
+	3650 1500 3250 1500
+Connection ~ 3250 1500
+Wire Wire Line
+	3150 3850 2550 3850
 $EndSCHEMATC

Commit message: zajecia
Parts:
- removed R3: 40k, Resistor_THT:R_Axial_DIN0207_L6.3mm_D2.5mm_P10.16mm_Horizontal, symbol Device:R
- removed R4: 10k, Resistor_THT:R_Axial_DIN0207_L6.3mm_D2.5mm_P10.16mm_Horizontal, symbol Device:R
- added RV1: R_POT_TRIM, Potentiometer_THT:Potentiometer_Piher_PT-10-V10_Vertical, symbol Device:R_POT_TRIM
- C3: value 10n -> 100n
- C4: footprint Capacitor_THT:C_Disc_D7.5mm_W5.0mm_P10.00mm -> Capacitor_SMD:C_0603_1608Metric_Pad1.05x0.95mm_HandSolder
Connections:
- net TRIG: now also RV1.2
- net at D2.1 (K): now also RV1.1
- net at D3.2 (A): now also RV1.3
Changed lines of the file:
@@
 	1    0    0    -1
 $EndComp
-Wire Wire Line
-	4150 4350 4450 4350
-Wire Wire Line
-	4150 4450 4150 4350
-Wire Wire Line
-	4150 4850 4150 4750
 $Comp
 L power:GND #PWR0103
@@
 $EndComp
 $Comp
-L Device:R R4
-U 1 1 5CB1EF33
-P 4150 4600
-F 0 "R4" H 4220 4646 50  0000 L CNN
-F 1 "10k" H 4220 4555 50  0000 L CNN
-F 2 "Resistor_THT:R_Axial_DIN0207_L6.3mm_D2.5mm_P10.16mm_Horizontal" V 4080 4600 50  0001 C CNN
-F 3 "~" H 4150 4600 50  0001 C CNN
-	1    4150 4600
-	1    0    0    -1
-$EndComp
-$Comp
-L Device:R R3
-U 1 1 5CB1E3D7
-P 4150 4100
-F 0 "R3" H 4220 4146 50  0000 L CNN
-F 1 "40k" H 4220 4055 50  0000 L CNN
-F 2 "Resistor_THT:R_Axial_DIN0207_L6.3mm_D2.5mm_P10.16mm_Horizontal" V 4080 4100 50  0001 C CNN
-F 3 "~" H 4150 4100 50  0001 C CNN
-	1    4150 4100
-	1    0    0    -1
-$EndComp
-$Comp
 L Device:C C4
 U 1 1 5CB1966A
@@
 F 0 "C4" H 3765 5396 50  0000 L CNN
 F 1 "820p" H 3765 5305 50  0000 L CNN
-F 2 "Capacitor_THT:C_Disc_D7.5mm_W5.0mm_P10.00mm" H 3688 5200 50  0001 C CNN
+F 2 "Capacitor_SMD:C_0603_1608Metric_Pad1.05x0.95mm_HandSolder" H 3688 5200 50  0001 C CNN
 F 3 "~" H 3650 5350 50  0001 C CNN
 	1    3650 5350
@@
 $EndComp
 Wire Wire Line
-	4150 3850 4150 3950
-Wire Wire Line
 	2850 5050 3650 5050
 Wire Wire Line
-	4150 4350 4150 4250
-Wire Wire Line
 	4450 4200 4650 4200
-Connection ~ 4150 4350
 Text Label 4650 4200 2    50   ~ 0
 TRIG
@@
 P 1300 5000
 F 0 "C3" H 1415 5046 50  0000 L CNN
-F 1 "10n" H 1415 4955 50  0000 L CNN
+F 1 "100n" H 1415 4955 50  0000 L CNN
 F 2 "Capacitor_THT:C_Disc_D7.5mm_W5.0mm_P10.00mm" H 1338 4850 50  0001 C CNN
 F 3 "~" H 1300 5000 50  0001 C CNN
@@
 	4150 3850 4050 3850
 Wire Wire Line
-	4450 4350 4450 4200
-Wire Wire Line
-	4450 4350 4450 4500
-Wire Wire Line
 	4450 4500 4650 4500
 Wire Wire Line
@@
 Wire Wire Line
 	4650 5050 3650 5050
-Connection ~ 4450 4350
 Connection ~ 3650 5050
 $Comp
@@
 Wire Wire Line
 	3150 3850 2550 3850
+Wire Wire Line
+	4450 4200 4450 4300
+$Comp
+L Device:R_POT_TRIM RV1
+U 1 1 5CDF9D06
+P 4150 4300
+F 0 "RV1" H 4080 4346 50  0000 R CNN
+F 1 "R_POT_TRIM" H 4080 4255 50  0000 R CNN
+F 2 "Potentiometer_THT:Potentiometer_Piher_PT-10-V10_Vertical" H 4150 4300 50  0001 C CNN
+F 3 "~" H 4150 4300 50  0001 C CNN
+	1    4150 4300
+	1    0    0    -1
+$EndComp
+Wire Wire Line
+	4300 4300 4450 4300
+Connection ~ 4450 4300
+Wire Wire Line
+	4450 4300 4450 4500
+Wire Wire Line
+	4150 3850 4150 4150
+Wire Wire Line
+	4150 4450 4150 4850
 $EndSCHEMATC

Commit message: wersja nie dzialajaca
Parts:
- C1: value 1u -> 22u
- U1: footprint Package_DIP:DIP-8_W7.62mm_LongPads -> Package_DIP:DIP-8_W10.16mm_LongPads
Connections:
- net GND: no longer J3.2 (Pin_2)
- net GNDCLK: now also J3.2 (Pin_2)
Changed lines of the file:
@@
-$EndComp
-$Comp
-L Device:C C1
-U 1 1 5CB0B470
-P 4100 1650
-F 0 "C1" H 4215 1696 50  0000 L CNN
-F 1 "1u" H 4215 1605 50  0000 L CNN
-F 2 "Capacitor_THT:CP_Axial_L11.0mm_D5.0mm_P18.00mm_Horizontal" H 4138 1500 50  0001 C CNN
-F 3 "~" H 4100 1650 50  0001 C CNN
-	1    4100 1650
-	1    0    0    -1
 $EndComp
 $Comp
@@
 F 0 "U1" H 2350 5431 50  0000 C CNN
 F 1 "NE555" H 2350 5340 50  0000 C CNN
-F 2 "Package_DIP:DIP-8_W7.62mm_LongPads" H 2350 4850 50  0001 C CNN
+F 2 "Package_DIP:DIP-8_W10.16mm_LongPads" H 2350 4850 50  0001 C CNN
 F 3 "http://www.ti.com/lit/ds/symlink/ne555.pdf" H 2350 4850 50  0001 C CNN
 	1    2350 4850
@@
 RST
 Wire Wire Line
-	2650 3600 2850 3600
-Wire Wire Line
 	1750 5050 1750 5350
 Wire Wire Line
@@
 Wire Wire Line
 	3600 4850 3750 4850
-$Comp
-L power:GND #PWR0102
-U 1 1 5CC493B4
-P 2850 3600
-F 0 "#PWR0102" H 2850 3350 50  0001 C CNN
-F 1 "GND" H 2855 3427 50  0000 C CNN
-F 2 "" H 2850 3600 50  0001 C CNN
-F 3 "" H 2850 3600 50  0001 C CNN
-	1    2850 3600
-	1    0    0    -1
-$EndComp
 $Comp
 L power:GND #PWR0106
@@
 Wire Wire Line
 	4150 4450 4150 4850
+$Comp
+L Device:C C1
+U 1 1 5CB0B470
+P 4100 1650
+F 0 "C1" H 4215 1696 50  0000 L CNN
+F 1 "22u" H 4215 1605 50  0000 L CNN
+F 2 "Capacitor_THT:CP_Axial_L11.0mm_D5.0mm_P18.00mm_Horizontal" H 4138 1500 50  0001 C CNN
+F 3 "~" H 4100 1650 50  0001 C CNN
+	1    4100 1650
+	1    0    0    -1
+$EndComp
+Text Label 2800 3700 0    50   ~ 0
+GNDCLK
+Wire Wire Line
+	2650 3600 2650 3700
+Wire Wire Line
+	2650 3700 2800 3700
 $EndSCHEMATC
