File: back/back.sch (KiCad schematic (older format))
At the start: 16 parts, among them J1 Screw_Terminal_01x02, J2 Screw_Terminal_01x02, J3 Screw_Terminal_01x02, Q1 IRF510, U1 NE555

Commit message: final 6.10
Parts:
- J1, J2, J3: footprint TerminalBlock_4Ucon:TerminalBlock_4Ucon_1x02_P3.50mm_Vertical -> TerminalBlock:TerminalBlock_bornier-2_P5.08mm
- L1: footprint back:ind_W60mm_D19mm_P38mm -> Footprints:ind_W60mm_D19mm_P38mm
Connections:
- net GND: no longer C3.2, C4.2
- net GNDCLK: now also C3.2, C4.2
Changed lines of the file:
@@
 EESchema Schematic File Version 4
 LIBS:back-cache
-EELAYER 29 0
+EELAYER 26 0
 EELAYER END
 $Descr A4 11693 8268
@@
 $EndComp
 $Comp
-L power:GND #PWR0103
-U 1 1 5CB2275D
-P 3650 5650
-F 0 "#PWR0103" H 3650 5400 50  0001 C CNN
-F 1 "GND" H 3655 5477 50  0000 C CNN
-F 2 "" H 3650 5650 50  0001 C CNN
-F 3 "" H 3650 5650 50  0001 C CNN
-	1    3650 5650
-	1    0    0    -1
-$EndComp
-$Comp
 L Device:C C4
 U 1 1 5CB1966A
@@
 Wire Wire Line
 	1850 4850 1300 4850
-$Comp
-L power:GND #PWR0104
-U 1 1 5CB39283
-P 1300 5300
-F 0 "#PWR0104" H 1300 5050 50  0001 C CNN
-F 1 "GND" H 1305 5127 50  0000 C CNN
-F 2 "" H 1300 5300 50  0001 C CNN
-F 3 "" H 1300 5300 50  0001 C CNN
-	1    1300 5300
-	1    0    0    -1
-$EndComp
 Wire Wire Line
 	1300 5150 1300 5300
@@
 F 0 "L1" V 3990 1400 50  0000 C CNN
 F 1 "400u" V 3899 1400 50  0000 C CNN
-F 2 "back:ind_W60mm_D19mm_P38mm" H 3800 1400 50  0001 C CNN
+F 2 "Footprints:ind_W60mm_D19mm_P38mm" H 3800 1400 50  0001 C CNN
 F 3 "~" H 3800 1400 50  0001 C CNN
 	1    3800 1400
@@
 F 0 "J2" H 5330 1592 50  0000 L CNN
 F 1 "Screw_Terminal_01x02" H 5330 1501 50  0000 L CNN
-F 2 "TerminalBlock_4Ucon:TerminalBlock_4Ucon_1x02_P3.50mm_Vertical" H 5250 1600 50  0001 C CNN
+F 2 "TerminalBlock:TerminalBlock_bornier-2_P5.08mm" H 5250 1600 50  0001 C CNN
 F 3 "~" H 5250 1600 50  0001 C CNN
 	1    5250 1600
@@
 F 0 "J1" H 1020 1275 50  0000 C CNN
 F 1 "Screw_Terminal_01x02" H 1020 1366 50  0000 C CNN
-F 2 "TerminalBlock_4Ucon:TerminalBlock_4Ucon_1x02_P3.50mm_Vertical" H 1100 1600 50  0001 C CNN
+F 2 "TerminalBlock:TerminalBlock_bornier-2_P5.08mm" H 1100 1600 50  0001 C CNN
 F 3 "~" H 1100 1600 50  0001 C CNN
 	1    1100 1600
@@
 F 0 "J3" V 2514 3212 50  0000 R CNN
 F 1 "Screw_Terminal_01x02" V 2423 3212 50  0000 R CNN
-F 2 "TerminalBlock_4Ucon:TerminalBlock_4Ucon_1x02_P3.50mm_Vertical" H 2550 3400 50  0001 C CNN
+F 2 "TerminalBlock:TerminalBlock_bornier-2_P5.08mm" H 2550 3400 50  0001 C CNN
 F 3 "~" H 2550 3400 50  0001 C CNN
 	1    2550 3400
@@
 Wire Wire Line
 	2650 3700 2800 3700
+Text Label 3650 5650 0    50   ~ 0
+GNDCLK
+Text Label 1300 5300 0    50   ~ 0
+GNDCLK
 $EndSCHEMATC
